File: Final_project_rbree.kicad_sch (KiCad schematic)
At the start: 44 parts, among them J1 Conn_01x02_Pin, J2 Conn_01x02_Pin, Q1 MMBT3904, Q3 AO3401A, U1 TL431, U2 LTV-817, U3 B1212, U4 2N7002, U7 NE555

Commit message: commit - final
Parts:
- added R22, R23: 1k, Resistor_SMD:R_0805_2012Metric_Pad1.20x1.40mm_HandSolder, symbol Device:R
Connections:
- net GND: now also R23.2
- net Vref: now also R22.2, R23.1; no longer C1.1, R1.1, R4.1, U1.3 (K)
- new net: C1.1, R1.1, R22.1, R4.1, U1.3 (K)
Changed lines of the file:
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@@
 	)
 	(junction
-		(at 92.71 179.07)
-		(diameter 0)
-		(color 0 0 0 0)
-	)
-	(junction
 		(at 224.79 207.01)
 		(diameter 0)
@@
 	)
 	(junction
+		(at 92.71 179.07)
+		(diameter 0)
+		(color 0 0 0 0)
+	)
+	(junction
 		(at 212.09 139.7)
 		(diameter 0)
@@
 	)
 	(junction
+		(at 127 179.07)
+		(diameter 0)
+		(color 0 0 0 0)
+	)
+	(junction
 		(at 358.14 106.68)
 		(diameter 0)
@@
 	(wire
 		(pts
-			(xy 212.09 128.27) (xy 212.09 129.54)
+			(xy 127 179.07) (xy 127 182.88)
 		)
 		(stroke
@@
 	(wire
 		(pts
-			(xy 241.3 85.09) (xy 276.86 85.09)
+			(xy 212.09 128.27) (xy 212.09 129.54)
 		)
 		(stroke
@@
 	(wire
 		(pts
-			(xy 72.39 107.95) (xy 73.66 107.95)
+			(xy 241.3 85.09) (xy 276.86 85.09)
 		)
 		(stroke
@@
 	(wire
 		(pts
-			(xy 224.79 109.22) (xy 224.79 101.6)
+			(xy 72.39 107.95) (xy 73.66 107.95)
 		)
 		(stroke
@@
 	(wire
 		(pts
-			(xy 236.22 195.58) (xy 247.65 195.58)
+			(xy 224.79 109.22) (xy 224.79 101.6)
 		)
 		(stroke
@@
 	(wire
 		(pts
-			(xy 92.71 179.07) (xy 127 179.07)
+			(xy 236.22 195.58) (xy 247.65 195.58)
 		)
 		(stroke
@@
 	(wire
 		(pts
+			(xy 120.65 179.07) (xy 127 179.07)
+		)
+		(stroke
+			(width 0)
+			(type default)
+		)
+	)
+	(wire
+		(pts
 			(xy 312.42 99.06) (xy 289.56 99.06)
 		)
@@
 	(wire
 		(pts
+			(xy 92.71 179.07) (xy 113.03 179.07)
+		)
+		(stroke
+			(width 0)
+			(type default)
+		)
+	)
+	(wire
+		(pts
 			(xy 67.31 138.43) (xy 72.39 138.43)
 		)
@@
 	(wire
 		(pts
+			(xy 127 190.5) (xy 127 205.74)
+		)
+		(stroke
+			(width 0)
+			(type default)
+		)
+	)
+	(wire
+		(pts
 			(xy 166.37 128.27) (xy 177.8 128.27)
 		)
@@
 		)
 	)
-	(label "Vin"
-		(at 111.76 128.27 0)
+	(label "Vref"
+		(at 127 175.26 0)
 		(fields_autoplaced yes)
 		(effects
 			(font
-				(size 1.27 1.27)
-				(thickness 0.254)
-				(bold yes)
+				(size 2.0066 2.0066)
 			)
 			(justify left bottom)
 		)
 	)
-	(label "Vref"
-		(at 100.33 179.07 0)
+	(label "Vin"
+		(at 111.76 128.27 0)
 		(fields_autoplaced yes)
 		(effects
@@
 	)
 	(symbol
+		(lib_id "Device:R")
+		(at 127 186.69 0)
+		(unit 1)
+		(exclude_from_sim no)
+		(in_bom yes)
+		(on_board yes)
+		(dnp no)
+		(fields_autoplaced yes)
+		(property "Reference" "R23"
+			(at 129.54 185.4199 0)
+			(effects
+				(font
+					(size 1.27 1.27)
+				)
+				(justify left)
+			)
+		)
+		(property "Value" "1k"
+			(at 129.54 187.9599 0)
+			(effects
+				(font
+					(size 1.27 1.27)
+				)
+				(justify left)
+			)
+		)
+		(property "Footprint" "Resistor_SMD:R_0805_2012Metric_Pad1.20x1.40mm_HandSolder"
+			(at 125.222 186.69 90)
+			(effects
+				(font
+					(size 1.27 1.27)
+				)
+				(hide yes)
+			)
+		)
+		(property "Datasheet" "~"
+			(at 127 186.69 0)
+			(effects
+				(font
+					(size 1.27 1.27)
+				)
+				(hide yes)
+			)
+		)
+		(property "Description" "Resistor"
+			(at 127 186.69 0)
+			(effects
+				(font
+					(size 1.27 1.27)
+				)
+				(hide yes)
+			)
+		)
+		(pin "2"
+		)
+		(pin "1"
+		)
+		(instances
+			(project "Final_project_rbree"
+				(path "/94e47eea-ee3d-40f5-84ad-e3510a82a1d2"
+					(reference "R23")
+					(unit 1)
+				)
+			)
+		)
+	)
+	(symbol
 		(lib_id "Transistor_BJT:MMBT3904")
 		(at 325.12 99.06 0)
@@
 	)
 	(symbol
+		(lib_id "Device:R")
+		(at 116.84 179.07 90)
+		(unit 1)
+		(exclude_from_sim no)
+		(in_bom yes)
+		(on_board yes)
+		(dnp no)
+		(property "Reference" "R22"
+			(at 116.586 182.118 90)
+			(effects
+				(font
+					(size 1.27 1.27)
+				)
+			)
+		)
+		(property "Value" "1k"
+			(at 116.586 184.658 90)
+			(effects
+				(font
+					(size 1.27 1.27)
+				)
+			)
+		)
+		(property "Footprint" "Resistor_SMD:R_0805_2012Metric_Pad1.20x1.40mm_HandSolder"
+			(at 116.84 180.848 90)
+			(effects
+				(font
+					(size 1.27 1.27)
+				)
+				(hide yes)
+			)
+		)
+		(property "Datasheet" "~"
+			(at 116.84 179.07 0)
+			(effects
+				(font
+					(size 1.27 1.27)
+				)
+				(hide yes)
+			)
+		)
+		(property "Description" "Resistor"
+			(at 116.84 179.07 0)
+			(effects
+				(font
+					(size 1.27 1.27)
+				)
+				(hide yes)
+			)
+		)
+		(pin "1"
+		)
+		(pin "2"
+		)
+		(instances
+			(project "Final_project_rbree"
+				(path "/94e47eea-ee3d-40f5-84ad-e3510a82a1d2"
+					(reference "R22")
+					(unit 1)
+				)
+			)
+		)
+	)
+	(symbol
 		(lib_id "Timer:NE555D")
 		(at 276.86 104.14 0)
@@
 					(unit 1)
 				)
+			)
+		)
+	)
+	(symbol
+		(lib_id "power:GND")
+		(at 127 205.74 0)
+		(unit 1)
+		(exclude_from_sim no)
+		(in_bom yes)
+		(on_board yes)
+		(dnp no)
+		(property "Reference" "#PWR021"
+			(at 127 212.09 0)
+			(effects
+				(font
+					(size 1.27 1.27)
+				)
+				(hide yes)
+			)
+		)
+		(property "Value" "GND"
+			(at 127.127 210.1342 0)
+			(effects
+				(font
+					(size 1.27 1.27)
+				)
+			)
+		)
+		(property "Footprint" ""
+			(at 127 205.74 0)
+			(effects
+				(font
+					(size 1.27 1.27)
+				)
+				(hide yes)
+			)
+		)
+		(property "Datasheet" ""
+			(at 127 205.74 0)
+			(effects
+				(font
+					(size 1.27 1.27)
+				)
+				(hide yes)
+			)
+		)
+		(property "Description" ""
+			(at 127 205.74 0)
+			(effects
+				(font
+					(size 1.27 1.27)
+				)
+				(hide yes)
+			)
+		)
+		(pin "1"
+		)
+		(instances
+			(project "Final_project_rbree"
+				(path "/94e47eea-ee3d-40f5-84ad-e3510a82a1d2"
+					(reference "#PWR021")
+					(unit 1)
+				)
